File: PCAB/ESP8266_COMPLETO/ESP8266_COMPLETO.kicad_pcb (KiCad board)
At the start: 2 copper layers, 93 parts, among them J1 Screw_Terminal_01x04, J2 Screw_Terminal_01x03, J3 Screw_Terminal_01x03, J4 Screw_Terminal_01x03, J5 Screw_Terminal_01x03, J6 USB_B_Mini, K1 SANYOU_SRD_Form_C, K2 SANYOU_SRD_Form_C, K3 SANYOU_SRD_Form_C, K4 SANYOU_SRD_Form_C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

Commit message: Cambios
Parts:
- removed the C3 at (63.5, -299.7)
- removed the C3 at (62.2, -370.8)
- removed the D1 at (29.2, -301.0)
- removed the D1 at (27.9, -372.1)
- removed the D2 at (69.8, -351.8)
- removed the D2 at (68.6, -422.9)
- removed the D3 at (54.6, -332.7)
- removed the D3 at (53.3, -403.9)
- removed the D4 at (90.2, -308.6)
- removed the D4 at (88.9, -379.7)
- removed the D5 at (54.6, -308.6)
- removed the D5 at (53.3, -379.7)
- removed the D6 at (90.2, -332.7)
- removed the D6 at (88.9, -403.9)
- removed the J1 at (77.5, -349.2)
- removed the J1 at (76.2, -420.4)
- removed the J2 at (30.5, -348.0)
- removed the J2 at (29.2, -419.1)
- removed the J3 at (115.6, -313.7)
- removed the J3 at (114.3, -384.8)
- removed the J4 at (30.5, -323.9)
- removed the J4 at (29.2, -395.0)
- removed the J5 at (115.6, -337.8)
- removed the J5 at (114.3, -408.9)
- removed the J6 at (77.5, -302.3)
- removed the J6 at (76.2, -373.4)
- removed the K1 at (38.1, -342.9)
- removed the K1 at (36.8, -414.0)
- removed the K2 at (38.1, -318.8)
- removed the K2 at (36.8, -389.9)
- removed the K3 at (90.2, -318.8)
- removed the K3 at (88.9, -389.9)
- removed the K4 at (90.2, -342.9)
- removed the K4 at (88.9, -414.0)
- removed the Q1 at (39.4, -330.2)
- removed the Q1 at (38.1, -401.3)
- removed the Q2 at (105.4, -306.1)
- removed the Q2 at (104.1, -377.2)
- removed the Q3 at (39.4, -306.1)
- removed the Q3 at (38.1, -377.2)
- removed the Q4 at (105.4, -330.2)
- removed the Q4 at (104.1, -401.3)
- removed the R1 at (69.8, -307.3)
- removed the R1 at (68.6, -378.5)
- removed the R2 at (47.0, -328.9)
- removed the R2 at (45.7, -400.1)
- removed the R3 at (47.0, -304.8)
- removed the R3 at (45.7, -375.9)
- removed the R4 at (97.8, -304.8)
- removed the R4 at (96.5, -375.9)
- removed the R5 at (97.8, -328.9)
- removed the R5 at (96.5, -400.1)
- removed the R6 at (43.2, -301.0)
- removed the R6 at (41.9, -372.1)
- removed the R7 at (66.0, -346.7)
- removed the R7 at (64.8, -417.8)
- removed the SW1 at (66.0, -303.5)
- removed the SW1 at (64.8, -374.6)
- removed the U1 at (61.0, -336.6)
- removed the U1 at (59.7, -407.7)
- removed the U2 at (59.7, -348.0)
- removed the U2 at (58.4, -419.1)
Routing:
- net (no net): track 2693.8 -> 0.00 mm, vias 4 -> 0
- removed copper zone on F.Cu, net (none)
